File: schematic/SAMduino/external.sch (KiCad schematic (older format))
At the start: 16 parts, among them IC4 SST26VF064B-104V_SM, IC5 MCP2221-I_SL, IC6 MCP2542FD-E_SN, J5 Conn_01x02, J6 Screw_Terminal_01x02

Commit message: Changed MCP2221 RST connection
Removed some comments
Parts:
- added R20: 10k, Resistor_SMD:R_0603_1608Metric, symbol Device:R
Connections:
- net GND: now also C26.1; no longer C26.2
- net VCC3V3: now also C26.2, R20.1; no longer C26.1
- net NRST: no longer names the net of IC5.4 (~RST)
- net NRST: now also R20.2
Other:
- note removed: "Is this needed? or 100n instead?"
- moved on the sheet: C26, C28, D3, D4, IC5, R5, R6
Changed lines of the file:
@@
 L SamacSys_Parts:MCP2221-I_SL IC5
 U 1 1 616206CE
-P 2500 4550
-F 0 "IC5" H 3050 4815 50  0000 C CNN
-F 1 "MCP2221-I_SL" H 3050 4724 50  0000 C CNN
-F 2 "SamacSys_Parts:SOIC127P600X175-14N" H 3450 4650 50  0001 L CNN
-F 3 "" H 3450 4550 50  0001 L CNN
-F 4 "USB 2.0 to I2C/UART Converter GPIO SO14 Microchip MCP2221-I/SL, USB Converter, USB 2.0 at 12Mbit/s, 3  5.5 V, 14-Pin SOIC" H 3450 4450 50  0001 L CNN "Description"
-F 5 "1.75" H 3450 4350 50  0001 L CNN "Height"
-F 6 "579-MCP2221-I/SL" H 3450 4250 50  0001 L CNN "Mouser Part Number"
-F 7 "https://www.mouser.co.uk/ProductDetail/Microchip-Technology/MCP2221-I-SL?qs=wzzOUr4NhYrXnl%252BgbTV6ag%3D%3D" H 3450 4150 50  0001 L CNN "Mouser Price/Stock"
-F 8 "Microchip" H 3450 4050 50  0001 L CNN "Manufacturer_Name"
-F 9 "MCP2221-I/SL" H 3450 3950 50  0001 L CNN "Manufacturer_Part_Number"
-	1    2500 4550
+P 2750 5200
+F 0 "IC5" H 3300 5465 50  0000 C CNN
+F 1 "MCP2221-I_SL" H 3300 5374 50  0000 C CNN
+F 2 "SamacSys_Parts:SOIC127P600X175-14N" H 3700 5300 50  0001 L CNN
+F 3 "" H 3700 5200 50  0001 L CNN
+F 4 "USB 2.0 to I2C/UART Converter GPIO SO14 Microchip MCP2221-I/SL, USB Converter, USB 2.0 at 12Mbit/s, 3  5.5 V, 14-Pin SOIC" H 3700 5100 50  0001 L CNN "Description"
+F 5 "1.75" H 3700 5000 50  0001 L CNN "Height"
+F 6 "579-MCP2221-I/SL" H 3700 4900 50  0001 L CNN "Mouser Part Number"
+F 7 "https://www.mouser.co.uk/ProductDetail/Microchip-Technology/MCP2221-I-SL?qs=wzzOUr4NhYrXnl%252BgbTV6ag%3D%3D" H 3700 4800 50  0001 L CNN "Mouser Price/Stock"
+F 8 "Microchip" H 3700 4700 50  0001 L CNN "Manufacturer_Name"
+F 9 "MCP2221-I/SL" H 3700 4600 50  0001 L CNN "Manufacturer_Part_Number"
+	1    2750 5200
 	1    0    0    -1
 $EndComp
@@
 L Device:C C28
 U 1 1 616AABD0
-P 4150 5300
-F 0 "C28" H 4265 5346 50  0000 L CNN
-F 1 "220n" H 4265 5255 50  0000 L CNN
-F 2 "Capacitor_SMD:C_0603_1608Metric" H 4188 5150 50  0001 C CNN
-F 3 "~" H 4150 5300 50  0001 C CNN
-	1    4150 5300
+P 4400 5950
+F 0 "C28" H 4515 5996 50  0000 L CNN
+F 1 "220n" H 4515 5905 50  0000 L CNN
+F 2 "Capacitor_SMD:C_0603_1608Metric" H 4438 5800 50  0001 C CNN
+F 3 "~" H 4400 5950 50  0001 C CNN
+	1    4400 5950
 	1    0    0    -1
 $EndComp
@@
 L Device:C C26
 U 1 1 616ABA21
-P 1950 4550
-F 0 "C26" V 1698 4550 50  0000 C CNN
-F 1 "100n" V 1789 4550 50  0000 C CNN
-F 2 "Capacitor_SMD:C_0603_1608Metric" H 1988 4400 50  0001 C CNN
-F 3 "~" H 1950 4550 50  0001 C CNN
-	1    1950 4550
-	0    1    1    0
+P 2450 4700
+F 0 "C26" V 2198 4700 50  0000 C CNN
+F 1 "100n" V 2289 4700 50  0000 C CNN
+F 2 "Capacitor_SMD:C_0603_1608Metric" H 2488 4550 50  0001 C CNN
+F 3 "~" H 2450 4700 50  0001 C CNN
+	1    2450 4700
+	-1   0    0    1
 $EndComp
 $Comp
 L Device:R R5
 U 1 1 616AC1B1
-P 1800 5650
-F 0 "R5" H 1870 5696 50  0000 L CNN
-F 1 "220R" H 1870 5605 50  0000 L CNN
-F 2 "Resistor_SMD:R_0603_1608Metric" V 1730 5650 50  0001 C CNN
-F 3 "~" H 1800 5650 50  0001 C CNN
-	1    1800 5650
+P 2050 6300
+F 0 "R5" H 2120 6346 50  0000 L CNN
+F 1 "220R" H 2120 6255 50  0000 L CNN
+F 2 "Resistor_SMD:R_0603_1608Metric" V 1980 6300 50  0001 C CNN
+F 3 "~" H 2050 6300 50  0001 C CNN
+	1    2050 6300
 	1    0    0    -1
 $EndComp
@@
 L Device:R R6
 U 1 1 616AC7F4
-P 2200 5650
-F 0 "R6" H 2270 5696 50  0000 L CNN
-F 1 "220R" H 2270 5605 50  0000 L CNN
-F 2 "Resistor_SMD:R_0603_1608Metric" V 2130 5650 50  0001 C CNN
-F 3 "~" H 2200 5650 50  0001 C CNN
-	1    2200 5650
+P 2450 6300
+F 0 "R6" H 2520 6346 50  0000 L CNN
+F 1 "220R" H 2520 6255 50  0000 L CNN
+F 2 "Resistor_SMD:R_0603_1608Metric" V 2380 6300 50  0001 C CNN
+F 3 "~" H 2450 6300 50  0001 C CNN
+	1    2450 6300
 	1    0    0    -1
 $EndComp
@@
 L Device:LED D3
 U 1 1 616AD36C
-P 1800 6150
-F 0 "D3" V 1747 6230 50  0000 L CNN
-F 1 "Green" V 1838 6230 50  0000 L CNN
-F 2 "LED_SMD:LED_0603_1608Metric" H 1800 6150 50  0001 C CNN
-F 3 "~" H 1800 6150 50  0001 C CNN
-	1    1800 6150
+P 2050 6800
+F 0 "D3" V 1997 6880 50  0000 L CNN
+F 1 "Green" V 2088 6880 50  0000 L CNN
+F 2 "LED_SMD:LED_0603_1608Metric" H 2050 6800 50  0001 C CNN
+F 3 "~" H 2050 6800 50  0001 C CNN
+	1    2050 6800
 	0    1    1    0
 $EndComp
@@
 L Device:LED D4
 U 1 1 616ADE58
-P 2200 6150
-F 0 "D4" V 2147 6230 50  0000 L CNN
-F 1 "Yellow" V 2238 6230 50  0000 L CNN
-F 2 "LED_SMD:LED_0603_1608Metric" H 2200 6150 50  0001 C CNN
-F 3 "~" H 2200 6150 50  0001 C CNN
-	1    2200 6150
+P 2450 6800
+F 0 "D4" V 2397 6880 50  0000 L CNN
+F 1 "Yellow" V 2488 6880 50  0000 L CNN
+F 2 "LED_SMD:LED_0603_1608Metric" H 2450 6800 50  0001 C CNN
+F 3 "~" H 2450 6800 50  0001 C CNN
+	1    2450 6800
 	0    1    1    0
 $EndComp
 Wire Wire Line
-	3600 4850 4150 4850
+	3850 5500 4400 5500
 $Comp
 L power:GND #PWR035
 U 1 1 616B00B3
-P 4150 5450
-F 0 "#PWR035" H 4150 5200 50  0001 C CNN
-F 1 "GND" H 4155 5277 50  0000 C CNN
-F 2 "" H 4150 5450 50  0001 C CNN
-F 3 "" H 4150 5450 50  0001 C CNN
-	1    4150 5450
+P 4400 6100
+F 0 "#PWR035" H 4400 5850 50  0001 C CNN
+F 1 "GND" H 4405 5927 50  0000 C CNN
+F 2 "" H 4400 6100 50  0001 C CNN
+F 3 "" H 4400 6100 50  0001 C CNN
+	1    4400 6100
 	1    0    0    -1
 $EndComp
@@
 L power:GND #PWR032
 U 1 1 616B0724
-P 1800 4550
-F 0 "#PWR032" H 1800 4300 50  0001 C CNN
-F 1 "GND" H 1805 4377 50  0000 C CNN
-F 2 "" H 1800 4550 50  0001 C CNN
-F 3 "" H 1800 4550 50  0001 C CNN
-	1    1800 4550
+P 2450 4850
+F 0 "#PWR032" H 2450 4600 50  0001 C CNN
+F 1 "GND" H 2455 4677 50  0000 C CNN
+F 2 "" H 2450 4850 50  0001 C CNN
+F 3 "" H 2450 4850 50  0001 C CNN
+	1    2450 4850
 	1    0    0    -1
 $EndComp
@@
 L power:GND #PWR033
 U 1 1 616B0DF5
-P 3700 4550
-F 0 "#PWR033" H 3700 4300 50  0001 C CNN
-F 1 "GND" V 3705 4422 50  0000 R CNN
-F 2 "" H 3700 4550 50  0001 C CNN
-F 3 "" H 3700 4550 50  0001 C CNN
-	1    3700 4550
+P 3950 5200
+F 0 "#PWR033" H 3950 4950 50  0001 C CNN
+F 1 "GND" V 3955 5072 50  0000 R CNN
+F 2 "" H 3950 5200 50  0001 C CNN
+F 3 "" H 3950 5200 50  0001 C CNN
+	1    3950 5200
 	0    -1   -1   0
 $EndComp
 Wire Wire Line
-	2100 4550 2250 4550
-Wire Wire Line
-	2500 4650 2100 4650
-Wire Wire Line
-	2100 4650 2100 5200
-Wire Wire Line
-	2100 5200 1800 5200
-Wire Wire Line
-	1800 5200 1800 5500
-Wire Wire Line
-	2500 4750 2200 4750
-Wire Wire Line
-	2200 4750 2200 5500
-Wire Wire Line
-	2200 5800 2200 6000
-Wire Wire Line
-	1800 5800 1800 6000
-Text GLabel 2600 6400 2    50   Input ~ 0
-VCC3V3
-Wire Wire Line
-	1800 6300 1800 6400
-Wire Wire Line
-	1800 6400 2200 6400
-Wire Wire Line
-	2200 6300 2200 6400
-Connection ~ 2200 6400
-Wire Wire Line
-	2200 6400 2600 6400
-Wire Wire Line
-	3700 4550 3600 4550
-Text GLabel 2250 4400 1    50   Input ~ 0
-VCC3V3
-Wire Wire Line
-	2250 4400 2250 4550
-Connection ~ 2250 4550
-Wire Wire Line
-	2250 4550 2500 4550
-Text GLabel 4350 4650 2    50   Input ~ 0
+	2750 5300 2350 5300
+Wire Wire Line
+	2350 5300 2350 5850
+Wire Wire Line
+	2350 5850 2050 5850
+Wire Wire Line
+	2050 5850 2050 6150
+Wire Wire Line
+	2750 5400 2450 5400
+Wire Wire Line
+	2450 5400 2450 6150
+Wire Wire Line
+	2450 6450 2450 6650
+Wire Wire Line
+	2050 6450 2050 6650
+Text GLabel 2850 7050 2    50   Input ~ 0
+VCC3V3
+Wire Wire Line
+	2050 6950 2050 7050
+Wire Wire Line
+	2050 7050 2450 7050
+Wire Wire Line
+	2450 6950 2450 7050
+Connection ~ 2450 7050
+Wire Wire Line
+	2450 7050 2850 7050
+Wire Wire Line
+	3950 5200 3850 5200
+Text GLabel 2200 4450 1    50   Input ~ 0
+VCC3V3
+Text GLabel 4600 5300 2    50   Input ~ 0
 Serial_D+
-Text GLabel 4350 4750 2    50   Input ~ 0
+Text GLabel 4600 5400 2    50   Input ~ 0
 Serial_D-
 Wire Wire Line
-	3600 4650 4350 4650
-Wire Wire Line
-	4350 4750 3600 4750
-Text GLabel 1350 4850 0    50   Input ~ 0
-NRST
-Text GLabel 1350 5050 0    50   Input ~ 0
+	3850 5300 4600 5300
+Wire Wire Line
+	4600 5400 3850 5400
+Text GLabel 1600 5700 0    50   Input ~ 0
 URXD0
-Text GLabel 1350 4950 0    50   Input ~ 0
+Text GLabel 1600 5600 0    50   Input ~ 0
 UTXD0
 Wire Wire Line
-	1350 4950 2500 4950
-Wire Wire Line
-	1350 5050 2500 5050
+	1600 5600 2750 5600
+Wire Wire Line
+	1600 5700 2750 5700
 $Comp
 L power:GND #PWR031
@@
 Text Notes 7400 2500 0    50   ~ 0
 CAN Transceiver
-Text Notes 2650 5450 0    50   ~ 0
+Text Notes 2900 6100 0    50   ~ 0
 USB to Serial Bridge
 Text Notes 2000 2650 0    50   ~ 0
@@
 Wire Wire Line
 	1650 1500 1650 1400
-Wire Wire Line
-	1350 4850 2500 4850
-NoConn ~ 2500 5150
-NoConn ~ 3600 4950
-NoConn ~ 3600 5050
-NoConn ~ 3600 5150
+NoConn ~ 2750 5800
+NoConn ~ 3850 5600
+NoConn ~ 3850 5700
+NoConn ~ 3850 5800
 $Comp
 L Connector:Screw_Terminal_01x02 J6
@@
 	1    0    0    -1
 $EndComp
-Text GLabel 4250 5000 2    50   Input ~ 0
-VCC3V3
-Wire Wire Line
-	4150 4850 4150 5000
-Wire Wire Line
-	4250 5000 4150 5000
-Connection ~ 4150 5000
-Wire Wire Line
-	4150 5000 4150 5150
-Text Notes 4500 5300 0    50   ~ 0
-Is this needed?  or 100n instead?
-Text Notes 1350 6200 0    50   ~ 0
+Text GLabel 4500 5650 2    50   Input ~ 0
+VCC3V3
+Wire Wire Line
+	4400 5500 4400 5650
+Wire Wire Line
+	4500 5650 4400 5650
+Connection ~ 4400 5650
+Wire Wire Line
+	4400 5650 4400 5800
+Text Notes 1600 6850 0    50   ~ 0
 MCU Tx\nindicator
-Text Notes 2550 6200 0    50   ~ 0
+Text Notes 2800 6850 0    50   ~ 0
 MCU Rx\nindicator
+$Comp
+L Device:R R20
+U 1 1 616A637E
+P 1800 5350
+F 0 "R20" H 1870 5396 50  0000 L CNN
+F 1 "10k" H 1870 5305 50  0000 L CNN
+F 2 "Resistor_SMD:R_0603_1608Metric" V 1730 5350 50  0001 C CNN
+F 3 "~" H 1800 5350 50  0001 C CNN
+	1    1800 5350
+	1    0    0    -1
+$EndComp
+Wire Wire Line
+	2750 5500 1800 5500
+Wire Wire Line
+	2750 5200 2200 5200
+Wire Wire Line
+	2200 5200 2200 4550
+Wire Wire Line
+	2450 4550 2200 4550
+Connection ~ 2200 4550
+Wire Wire Line
+	2200 4550 2200 4450
+Wire Wire Line
+	1800 5200 2200 5200
+Connection ~ 2200 5200
 $EndSCHEMATC

Commit message: PCB routed - needs optimization
Connections:
- net at IC6.6 (CANL), R7.2: now also J6.1 (Pin_1); no longer J6.2 (Pin_2)
- net at IC6.7 (CANH), J5.2 (Pin_2): now also J6.2 (Pin_2); no longer J6.1 (Pin_1)
Changed lines of the file:
@@
 L Connector:Screw_Terminal_01x02 J6
 U 1 1 616DF8B0
-P 9450 1950
-F 0 "J6" H 9530 1896 50  0000 L CNN
-F 1 "Screw_Terminal_01x02" H 9530 1851 50  0001 L CNN
-F 2 "SamacSys_Parts:1725656" H 9450 1950 50  0001 C CNN
-F 3 "~" H 9450 1950 50  0001 C CNN
-	1    9450 1950
-	1    0    0    -1
+P 9450 2050
+F 0 "J6" H 9530 1996 50  0000 L CNN
+F 1 "Screw_Terminal_01x02" H 9530 1951 50  0001 L CNN
+F 2 "SamacSys_Parts:1725656" H 9450 2050 50  0001 C CNN
+F 3 "~" H 9450 2050 50  0001 C CNN
+	1    9450 2050
+	1    0    0    1
 $EndComp
 Text GLabel 4500 5650 2    50   Input ~ 0
